File: SubSequence.kicad_pcb (KiCad board)
At the start: 2 copper layers, 80.3 x 100 mm, 50 parts, among them J1 Conn_02x03_Odd_Even, J2 Conn_02x03_Odd_Even, J3 Conn_01x03, SW1 SW_Push, SW2 SW_SPDT_MSM, SW3 SW_SPDT_MSM, SW4 SW_SPDT_MSM, SW5 SW_SPDT_MSM, SW6 SW_SPDT_MSM, SW7 SW_SPDT_MSM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

Commit message: Finished layout.
Parts:
- moved R1 0.97 mm to (152.4, 132.1), turned to 90 degrees
- moved SW1 0.69 mm to (150.1, 135.3)
- moved SW3 0.38 mm to (142.2, 86.4)
- moved SW4 0.25 mm to (121.8, 104.0)
- moved SW7 0.15 mm to (182.9, 104.1)
Connections:
- C1 pad 2: (no net) -> GND
- C2 pad 1: (no net) -> GND
- C3 pad 1: (no net) -> GND
- C4 pad 2: (no net) -> GND
- J1 pad 1: (no net) -> GND
- J1 pad 2: (no net) -> GND
- J2 pad 6: (no net) -> GND
- J3 pad 1: (no net) -> GND
- RV1 pad 3: (no net) -> GND
- RV2 pad 3: (no net) -> GND
- RV3 pad 3: (no net) -> GND
- RV4 pad 3: (no net) -> GND
- RV5 pad 3: (no net) -> GND
- RV6 pad 3: (no net) -> GND
- RV7 pad 3: (no net) -> GND
- RV8 pad 3: (no net) -> GND
- SW1 pad 2: (no net) -> GND
- U1 pad 21: (no net) -> GND
- U1 pad 5: (no net) -> GND
Routing:
- net +5V: track 0.00 -> 337.1 mm, vias 0 -> 10
- net /MCU328/PB1: track 0.00 -> 216.7 mm, vias 0 -> 6
- net /MCU328/PB2: track 0.00 -> 195.9 mm, vias 0 -> 4
- net /MCU328/PD2: track 0.00 -> 178.5 mm, vias 0 -> 10
- net Net-(D15-Pad2): track 0.00 -> 58.4 mm, vias 0 -> 2
- net Net-(D9-Pad2): track 0.00 -> 41.7 mm, vias 0 -> 2
- net Net-(D14-Pad2): track 0.00 -> 41.1 mm
- net SCL: track 0.00 -> 35.9 mm
- net SDA: track 0.00 -> 35.9 mm
- net Net-(D16-Pad2): track 0.00 -> 34.1 mm
- net Net-(D11-Pad2): track 0.00 -> 33.3 mm
- net Net-(D13-Pad2): track 0.00 -> 33.2 mm
- net Net-(D12-Pad2): track 0.00 -> 30.4 mm
- net Net-(J2-Pad5): track 71.0 -> 100.3 mm
- net Net-(D10-Pad2): track 0.00 -> 28.6 mm
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- added copper zone on B.Cu, net GND
- added copper zone on F.Cu, net GND

Commit message: Silk-screens.
Other:
- board text added: "Rev A"
- board text added: "SubSequence"
- board text added: "© Marangisto 2018"
