File: SubSequence.kicad_pcb (KiCad board)
At the start: 2 copper layers, 80.3 x 100 mm, 50 parts, among them J1 Conn_02x03_Odd_Even, J2 Conn_02x03_Odd_Even, J3 Conn_01x03, SW1 SW_Push, SW2 SW_SPDT_MSM, SW3 SW_SPDT_MSM, SW4 SW_SPDT_MSM, SW5 SW_SPDT_MSM, SW6 SW_SPDT_MSM, SW7 SW_SPDT_MSM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

Commit message: Added pull-up resistors.
Parts:
- added R10: 10k, Resistor_SMD:R_0805_2012Metric, B.Cu at (149.4, 78.7)
- added R11: 10k, Resistor_SMD:R_0805_2012Metric, B.Cu at (182.9, 121.4)
Routing:
- net /MCU328/PB1: track 216.7 -> 228.4 mm
- net +5V: track 337.1 -> 348.7 mm
- net /MCU328/PD2: track 178.5 -> 180.8 mm
- net /MCU328/PB6: track 29.3 -> 30.7 mm
- net GND: vias 11 -> 12
Changed lines of the file:
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@@
-(kicad_pcb (version 20171130) (host pcbnew 5.0.0-fee4fd1~66~ubuntu16.04.1)
+(kicad_pcb (version 20171130) (host pcbnew "(5.0.1-3-g963ef8bb5)")
   (general
     (thickness 1.6)
     (drawings 37)
-    (tracks 673)
+    (tracks 687)
     (zones 0)
-    (modules 50)
+    (modules 52)
     (nets 47)
   )
@@
     (pad_drill 0.762)
     (pad_to_mask_clearance 0.2)
+    (solder_mask_min_width 0.25)
     (aux_axis_origin 0 0)
     (visible_elements FFFFFF7F)
@@
     (add_net SCL)
     (add_net SDA)
+  )
+  (module Resistor_SMD:R_0805_2012Metric (layer B.Cu)
+    (at 149.352 78.74 270)
+    (descr "Resistor SMD 0805 (2012 Metric), square (rectangular) end terminal, IPC_7351 nominal, (Body size source: https://docs.google.com/spreadsheets/d/1BsfQQcO9C6DZCsRaXUlFlo91Tg2WpOkGARC1WS5S8t0/edit?usp=sharing), generated with kicad-footprint-generator")
+    (tags resistor)
+    (attr smd)
+    (fp_text reference R10 (at 0 -2.032 270) (layer B.SilkS)
+      (effects (font (size 1 1) (thickness 0.15)) (justify mirror))
+    )
+    (fp_text value 10k (at 0 -1.65 270) (layer B.Fab)
+      (effects (font (size 1 1) (thickness 0.15)) (justify mirror))
+    )
+    (fp_text user %R (at 0 0 270) (layer B.Fab)
+      (effects (font (size 0.5 0.5) (thickness 0.08)) (justify mirror))
+    )
+    (fp_line (start 1.68 -0.95) (end -1.68 -0.95) (layer B.CrtYd) (width 0.05))
+    (fp_line (start 1.68 0.95) (end 1.68 -0.95) (layer B.CrtYd) (width 0.05))
+    (fp_line (start -1.68 0.95) (end 1.68 0.95) (layer B.CrtYd) (width 0.05))
+    (fp_line (start -1.68 -0.95) (end -1.68 0.95) (layer B.CrtYd) (width 0.05))
+    (fp_line (start -0.258578 -0.71) (end 0.258578 -0.71) (layer B.SilkS) (width 0.12))
+    (fp_line (start -0.258578 0.71) (end 0.258578 0.71) (layer B.SilkS) (width 0.12))
+    (fp_line (start 1 -0.6) (end -1 -0.6) (layer B.Fab) (width 0.1))
+    (fp_line (start 1 0.6) (end 1 -0.6) (layer B.Fab) (width 0.1))
+    (fp_line (start -1 0.6) (end 1 0.6) (layer B.Fab) (width 0.1))
+    (fp_line (start -1 -0.6) (end -1 0.6) (layer B.Fab) (width 0.1))
+    (pad 2 smd roundrect (at 0.9375 0 270) (size 0.975 1.4) (layers B.Cu B.Paste B.Mask) (roundrect_rratio 0.25)
+      (net 42 /MCU328/PD2))
+    (pad 1 smd roundrect (at -0.9375 0 270) (size 0.975 1.4) (layers B.Cu B.Paste B.Mask) (roundrect_rratio 0.25)
+      (net 2 +5V))
+    (model ${KISYS3DMOD}/Resistor_SMD.3dshapes/R_0805_2012Metric.wrl
+      (at (xyz 0 0 0))
+      (scale (xyz 1 1 1))
+      (rotate (xyz 0 0 0))
+    )
+  )
+  (module Resistor_SMD:R_0805_2012Metric (layer B.Cu)
+    (at 182.88 121.412 90)
+    (descr "Resistor SMD 0805 (2012 Metric), square (rectangular) end terminal, IPC_7351 nominal, (Body size source: https://docs.google.com/spreadsheets/d/1BsfQQcO9C6DZCsRaXUlFlo91Tg2WpOkGARC1WS5S8t0/edit?usp=sharing), generated with kicad-footprint-generator")
+    (tags resistor)
+    (attr smd)
+    (fp_text reference R11 (at 0 1.65 90) (layer B.SilkS)
+      (effects (font (size 1 1) (thickness 0.15)) (justify mirror))
+    )
+    (fp_text value 10k (at 0 -1.65 90) (layer B.Fab)
+      (effects (font (size 1 1) (thickness 0.15)) (justify mirror))
+    )
+    (fp_line (start -1 -0.6) (end -1 0.6) (layer B.Fab) (width 0.1))
+    (fp_line (start -1 0.6) (end 1 0.6) (layer B.Fab) (width 0.1))
+    (fp_line (start 1 0.6) (end 1 -0.6) (layer B.Fab) (width 0.1))
+    (fp_line (start 1 -0.6) (end -1 -0.6) (layer B.Fab) (width 0.1))
+    (fp_line (start -0.258578 0.71) (end 0.258578 0.71) (layer B.SilkS) (width 0.12))
+    (fp_line (start -0.258578 -0.71) (end 0.258578 -0.71) (layer B.SilkS) (width 0.12))
+    (fp_line (start -1.68 -0.95) (end -1.68 0.95) (layer B.CrtYd) (width 0.05))
+    (fp_line (start -1.68 0.95) (end 1.68 0.95) (layer B.CrtYd) (width 0.05))
+    (fp_line (start 1.68 0.95) (end 1.68 -0.95) (layer B.CrtYd) (width 0.05))
+    (fp_line (start 1.68 -0.95) (end -1.68 -0.95) (layer B.CrtYd) (width 0.05))
+    (fp_text user %R (at 0 0 90) (layer B.Fab)
+      (effects (font (size 0.5 0.5) (thickness 0.08)) (justify mirror))
+    )
+    (pad 1 smd roundrect (at -0.9375 0 90) (size 0.975 1.4) (layers B.Cu B.Paste B.Mask) (roundrect_rratio 0.25)
+      (net 2 +5V))
+    (pad 2 smd roundrect (at 0.9375 0 90) (size 0.975 1.4) (layers B.Cu B.Paste B.Mask) (roundrect_rratio 0.25)
+      (net 43 /MCU328/PB1))
+    (model ${KISYS3DMOD}/Resistor_SMD.3dshapes/R_0805_2012Metric.wrl
+      (at (xyz 0 0 0))
+      (scale (xyz 1 1 1))
+      (rotate (xyz 0 0 0))
+    )
   )
   (module Buttons_Switches_THT:SW_PUSH_6mm_h9.5mm (layer F.Cu)
@@
   (via (at 149.86 95.758) (size 0.8) (drill 0.4) (layers F.Cu B.Cu) (net 2))
   (segment (start 152.4 76.454) (end 152.4 83.058) (width 0.75) (layer B.Cu) (net 2))
-  (segment (start 149.606 73.66) (end 152.4 76.454) (width 0.75) (layer B.Cu) (net 2))
   (segment (start 152.4 65.51) (end 151.914 65.51) (width 0.75) (layer B.Cu) (net 2))
   (segment (start 149.606 67.818) (end 149.606 73.66) (width 0.75) (layer B.Cu) (net 2))
   (segment (start 151.914 65.51) (end 149.606 67.818) (width 0.75) (layer B.Cu) (net 2))
+  (segment (start 149.352 76.454) (end 150.876 74.93) (width 0.25) (layer B.Cu) (net 2))
+  (segment (start 149.352 77.8025) (end 149.352 76.454) (width 0.25) (layer B.Cu) (net 2))
+  (segment (start 150.876 74.93) (end 152.4 76.454) (width 0.75) (layer B.Cu) (net 2))
+  (segment (start 149.606 73.66) (end 150.876 74.93) (width 0.75) (layer B.Cu) (net 2))
+  (segment (start 185.38 124.8495) (end 182.88 122.3495) (width 0.25) (layer B.Cu) (net 2))
+  (segment (start 185.38 129.42001) (end 185.38 124.8495) (width 0.25) (layer B.Cu) (net 2))
   (segment (start 186.69 70.612) (end 186.69 72.71) (width 0.25) (layer B.Cu) (net 3))
   (segment (start 188.976 68.326) (end 186.69 70.612) (width 0.25) (layer B.Cu) (net 3))
@@
   (segment (start 140.332 72.26) (end 138.43 72.26) (width 0.25) (layer B.Cu) (net 21))
   (segment (start 140.462 72.39) (end 140.332 72.26) (width 0.25) (layer B.Cu) (net 21))
-  (segment (start 150.172615 90.194188) (end 150.80901 90.830583) (width 0.25) (layer B.Cu) (net 21))
-  (segment (start 150.314029 90.052775) (end 150.172615 90.194188) (width 0.25) (layer B.Cu) (net 21))
-  (segment (start 149.606 88.138) (end 149.606 89.344746) (width 0.25) (layer B.Cu) (net 21))
-  (segment (start 149.606 89.344746) (end 150.314029 90.052775) (width 0.25) (layer B.Cu) (net 21))
-  (segment (start 143.39 72.39) (end 144.66 73.66) (width 0.25) (layer B.Cu) (net 21))
-  (segment (start 142.24 72.39) (end 143.39 72.39) (width 0.25) (layer B.Cu) (net 21))
-  (segment (start 144.66 73.66) (end 147.066 73.66) (width 0.25) (layer B.Cu) (net 21))
-  (segment (start 147.066 73.66) (end 151.13 77.724) (width 0.25) (layer B.Cu) (net 21))
-  (segment (start 151.13 77.724) (end 151.13 86.614) (width 0.25) (layer B.Cu) (net 21))
-  (segment (start 151.13 86.614) (end 149.606 88.138) (width 0.25) (layer B.Cu) (net 21))
+  (segment (start 143.39 72.39) (end 142.24 72.39) (width 0.25) (layer B.Cu) (net 21))
+  (segment (start 144.66 73.66) (end 143.39 72.39) (width 0.25) (layer B.Cu) (net 21))
+  (segment (start 150.314029 90.052775) (end 149.606 89.344746) (width 0.25) (layer B.Cu) (net 21))
+  (segment (start 147.574 74.168) (end 147.066 73.66) (width 0.25) (layer B.Cu) (net 21))
+  (segment (start 148.082 78.74) (end 147.574 78.232) (width 0.25) (layer B.Cu) (net 21))
+  (segment (start 150.368 78.74) (end 148.082 78.74) (width 0.25) (layer B.Cu) (net 21))
+  (segment (start 151.13 86.614) (end 151.13 79.502) (width 0.25) (layer B.Cu) (net 21))
+  (segment (start 149.606 88.138) (end 151.13 86.614) (width 0.25) (layer B.Cu) (net 21))
+  (segment (start 147.574 78.232) (end 147.574 74.168) (width 0.25) (layer B.Cu) (net 21))
+  (segment (start 147.066 73.66) (end 144.66 73.66) (width 0.25) (layer B.Cu) (net 21))
+  (segment (start 151.13 79.502) (end 150.368 78.74) (width 0.25) (layer B.Cu) (net 21))
+  (segment (start 149.606 89.344746) (end 149.606 88.138) (width 0.25) (layer B.Cu) (net 21))
+  (segment (start 150.172615 90.194188) (end 150.314029 90.052775) (width 0.25) (layer B.Cu) (net 21))
+  (segment (start 150.80901 90.830583) (end 150.172615 90.194188) (width 0.25) (layer B.Cu) (net 21))
   (segment (start 165.1 86.36) (end 162.56 86.36) (width 0.25) (layer B.Cu) (net 22))
   (segment (start 169.418 82.042) (end 165.1 86.36) (width 0.25) (layer B.Cu) (net 22))
@@
   (segment (start 137.668 89.916) (end 135.89 88.138) (width 0.25) (layer B.Cu) (net 42))
   (segment (start 137.668 92.837) (end 137.668 89.916) (width 0.25) (layer B.Cu) (net 42))
+  (segment (start 150.368 81.534) (end 149.352 80.518) (width 0.25) (layer B.Cu) (net 42))
+  (segment (start 149.352 80.518) (end 149.352 79.6775) (width 0.25) (layer B.Cu) (net 42))
   (segment (start 122.68 108.46) (end 121.838 108.46) (width 0.25) (layer B.Cu) (net 43))
   (segment (start 157.155686 91.06) (end 162.56 91.06) (width 0.25) (layer B.Cu) (net 43))
@@
   (segment (start 169.317 108.686) (end 182.88 108.686) (width 0.25) (layer B.Cu) (net 43))
   (segment (start 162.433 115.57) (end 169.317 108.686) (width 0.25) (layer B.Cu) (net 43))
+  (segment (start 182.88 119.887) (end 182.88 108.84) (width 0.25) (layer B.Cu) (net 43))
+  (segment (start 182.88 120.4745) (end 182.88 119.887) (width 0.25) (layer B.Cu) (net 43))
   (segment (start 182.88 72.39) (end 181.102 72.39) (width 0.25) (layer B.Cu) (net 44))
   (segment (start 180.972 72.26) (end 179.07 72.26) (width 0.25) (layer B.Cu) (net 44))
@@
   (via (at 176.911 104.267) (size 0.8) (drill 0.4) (layers F.Cu B.Cu) (net 46))
   (via (at 128.143 104.521) (size 0.8) (drill 0.4) (layers F.Cu B.Cu) (net 46))
+  (via (at 172.974 116.078) (size 0.8) (drill 0.4) (layers F.Cu B.Cu) (net 46))
   (zone (net 46) (net_name GND) (layer F.Cu) (hatch edge 0.508)
     (connect_pads (clearance 0.508))

Commit message: Added 3-d models (except toggle switches).
Parts:
- C1, C2, C3: footprint Capacitors_SMD:C_0805 -> Capacitor_SMD:C_0805_2012Metric
- C4: footprint Capacitors_SMD:CP_Elec_4x5.8 -> Capacitor_SMD:CP_Elec_4x5.8
- D1, D2, D3, D4, D5, D6, D7, D8: footprint LEDs:LED_D3.0mm -> LED_THT:LED_D3.0mm
- D10, D11, D12, D13, D14, D15, D16, D9: footprint Diodes_SMD:D_SOD-123F -> Diode_SMD:D_SOD-123F
- J1, J2: footprint Pin_Headers:Pin_Header_Straight_2x03_Pitch2.54mm -> Connector_PinHeader_2.54mm:PinHeader_2x03_P2.54mm_Vertical
- J3: footprint Pin_Headers:Pin_Header_Straight_1x03_Pitch2.54mm -> Connector_PinHeader_2.54mm:PinHeader_1x03_P2.54mm_Vertical
- R1, R2, R3, R4, R5, R6, R7, R8, R9: footprint Resistors_SMD:R_0805 -> Resistor_SMD:R_0805_2012Metric
- SW1: footprint Buttons_Switches_THT:SW_PUSH_6mm_h9.5mm -> Button_Switch_THT:SW_PUSH_6mm_H9.5mm
- U1: footprint Housings_QFP:TQFP-32_7x7mm_Pitch0.8mm -> Package_QFP:TQFP-32_7x7mm_P0.8mm
